Commit message: update

File: src/rm_nav_bringup/urdf/sentry_robot_sim.xacro (robot description, xacro)
@@ -18,5 +18,5 @@
     <visual>
       <geometry>
-        <box size="0.2 .3 .1"/>
+        <box size="0.3 0.5 0.1"/>
       </geometry>
       <origin rpy="0 0 ${PI/2}" xyz="0 0 0.05"/>
@@ -27,9 +27,9 @@
     <collision>
       <geometry>
-        <box size="0.2 .3 0.1"/>
+        <box size="0.2 .5 0.1"/>
       </geometry>
       <origin rpy="0 0 ${PI/2}" xyz="0 0 0.05"/>
     </collision>
-    <xacro:default_inertial mass="8.2"/>
+    <xacro:default_inertial mass="50.0"/>
   </link>
   <joint name="dummy_joint" type="fixed">
@@ -52,6 +52,6 @@
       </geometry>
     </collision>
-    <mu1>0.5</mu1>
-    <mu2>0.5</mu2>
+    <mu1>1.0</mu1>
+    <mu2>1.0</mu2>
     <xacro:default_inertial mass="0.5"/>
   </link>
@@ -160,5 +160,5 @@
       <mass value="1e-2" />
       <origin xyz="0 0 0" rpy="0 0 0"/>
-      <inertia ixx="1e-6" ixy="0" ixz="0" iyy="1e-6" iyz="0" izz="1e-6" />
+      <inertia ixx="1.0" ixy="0" ixz="0" iyy="1.0" iyz="0" izz="1.0" />
     </inertial>
   </link>
